File: GigaPower200V.kicad_pcb (KiCad board)
At the start: 4 copper layers, 50 x 20 mm, 70 parts, among them J1 Conn_02x10_Odd_Even, J2 Conn_02x10_Odd_Even, Q1 CPC3980, Q2 BSZ42DN25NS3G, Q3 MMBTA92, U2 TL494, U3 AP63356DV, U4 IR2181, U5 AP63356DV, U6 TL431

Commit message: initial
Parts:
- U3, U5: footprint GigaVescLibs:V-DFN3020-13_DIO -> X3.0CH-Library:V-DFN3020-13_DIO
- moved R26 5.06 mm to (160.8, 92.9), turned to -90 degrees
- moved D1 4.48 mm to (148.2, 99.4)
- moved R22 4.48 mm to (145.1, 98.9)
- moved C13 4.48 mm to (151.5, 101.3)
- moved C17 4.48 mm to (145.1, 101.1)
- moved R23 4.48 mm to (150.5, 101.3)
- moved R24 4.48 mm to (151.0, 102.8)
- moved R25 4.48 mm to (145.1, 100.0)
- moved U6 4.48 mm to (148.0, 102.1)
- moved D3 2.86 mm to (163.0, 102.2)
- moved R27 2.69 mm to (161.1, 90.9), turned to 45 degrees
- moved R21 2.28 mm to (159.6, 86.2)
- moved D7 2.21 mm to (163.2, 86.9)
- moved C16 2.20 mm to (159.6, 89.0)
- moved U4 2.20 mm to (154.8, 89.4)
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Routing:
- net VIN: track 13.1 -> 22.8 mm, vias 8 -> 6
- net GND: track 21.7 -> 26.3 mm, vias 31 -> 37
- net Net-(Q1-S): track 9.73 -> 7.06 mm
- net Net-(U2-FB): track 10.8 -> 12.6 mm
- net STARTUP: track 45.1 -> 46.7 mm
- net Net-(U2-E1): track 11.8 -> 10.3 mm
- net Net-(Q2-G): track 6.50 -> 5.24 mm
- net Net-(D3-K): track 13.5 -> 14.6 mm
- net Net-(D7-K): track 8.33 -> 9.31 mm
- net Net-(Q3-B): track 9.05 -> 8.43 mm
- net +5V: track 42.0 -> 42.5 mm
Other:
- board text added: "12V"
- board text added: "GigaESC by Kaminaris Power 200V V1.0.0"
- board text removed: "3.3R"
- board text removed: "F"
- board text removed: "GigaESC by Kaminaris Compute Module"
- board text removed: "R"
- board text removed: "R1"
- board text removed: "R2"
- board text removed: "R3"
- board text removed: "X3.0 SLOT"
