File: GigaPower200V.kicad_sch (KiCad schematic)
At the start: 70 parts, among them J1 Conn_02x10_Odd_Even, J2 Conn_02x10_Odd_Even, Q1 CPC3980, Q2 BSZ42DN25NS3G, Q3 MMBTA92, U2 TL494, U3 AP63356DV, U4 IR2181, U5 AP63356DV, U6 TL431

Commit message: initial
Parts:
- U3, U5: footprint GigaVescLibs:V-DFN3020-13_DIO -> X3.0CH-Library:V-DFN3020-13_DIO; symbol GigaVescSymbols:AP63357DV -> X3.0CH-Library:AP63357DV
- U6: symbol GigaESCSymbols:TL431 -> X3.0CH-Library:TL431
Other:
- note removed: "D2 Leg 1 is NC so we can use that to help with layout"
- moved on the sheet: C10, C11, C12, C13, C14, C15, C16, C17, C18, C20, C21, C22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
